File: Board - Copy_bsckup/uSATAboard.sch (KiCad schematic (older format))
At the start: 8 parts, among them CN1 USATA, P1 CONN_1, P2 CONN_1, P3 CONN_1, P4 CONN_1, P5 CONN_1, P6 CONN_1, P7 CONN_1

Commit message: to repeat
done
Parts:
- renumbered CN1 to CN2
Changed lines of the file:
@@
 LIBS:memory
 LIBS:xilinx
+LIBS:special
 LIBS:microcontrollers
 LIBS:dsp
@@
 LIBS:myLib
 LIBS:uSATAboard-cache
-EELAYER 25 0
+EELAYER 27 0
 EELAYER END
 $Descr A4 11693 8268
@@
 $EndDescr
 $Comp
-L USATA CN1
+L USATA CN2
 U 1 1 53E0E90C
 P 6800 2800
-F 0 "CN1" H 6800 2700 60  0000 C CNN
+F 0 "CN2" H 6800 2700 60  0000 C CNN
 F 1 "USATA" H 6800 2800 60  0000 C CNN
 F 2 "" H 6800 2800 60  0000 C CNN
