File: Board/uSATAboard.sch (KiCad schematic (older format))
At the start: 8 parts, among them CN2 USATA, P1 CONN_1, P2 CONN_1, P3 CONN_1, P4 CONN_1, P5 CONN_1, P6 CONN_1, P7 CONN_1

Commit message: to repeat
done
Parts:
- removed P1, P2, P3, P4, P5, P6, P7: CONN_1, symbol CONN_1
- added CN1: B+, symbol CONN1
- added CN2: B-, symbol CONN1
- added CN3, CN6: GND, symbol CONN1
- added CN4: A-, symbol CONN1
- added CN5: A+, symbol CONN1
- added CN7: +3.3V, symbol CONN1
- renumbered CN2 to CN8
Other:
- moved on the sheet: CN8
Changed lines of the file:
@@
 LIBS:memory
 LIBS:xilinx
-LIBS:special
 LIBS:microcontrollers
 LIBS:dsp
@@
 LIBS:contrib
 LIBS:valves
-LIBS:myLib
-LIBS:uSATAboard-cache
-EELAYER 27 0
+LIBS:eeepc_ssd
+EELAYER 25 0
 EELAYER END
 $Descr A4 11693 8268
@@
 $EndDescr
 $Comp
-L USATA CN2
+L USATA CN8
 U 1 1 53E0E90C
-P 6800 2800
-F 0 "CN2" H 6800 2700 60  0000 C CNN
-F 1 "USATA" H 6800 2800 60  0000 C CNN
-F 2 "" H 6800 2800 60  0000 C CNN
-F 3 "" H 6800 2800 60  0000 C CNN
-	1    6800 2800
+P 6800 3000
+F 0 "CN8" H 6875 3050 60  0000 C CNN
+F 1 "USATA" H 7325 1125 60  0000 C CNN
+F 2 "" H 6800 3000 60  0000 C CNN
+F 3 "" H 6800 3000 60  0000 C CNN
+	1    6800 3000
 	1    0    0    -1
 $EndComp
@@
 NoConn ~ 6500 4650
 NoConn ~ 6500 4750
-Text Label 6500 3050 2    60   ~ 0
+Text GLabel 6500 4150 0    60   Input ~ 0
 GND
-Text Label 6500 3150 2    60   ~ 0
+Text GLabel 6500 4050 0    60   Input ~ 0
+GND
+Text GLabel 6500 3650 0    60   Input ~ 0
+GND
+Text GLabel 6500 3350 0    60   Input ~ 0
+GND
+Text GLabel 6500 3050 0    60   Input ~ 0
+GND
+Text GLabel 6500 3150 0    60   Input ~ 0
 A+
-Text Label 6500 3250 2    60   ~ 0
+Text GLabel 6500 3250 0    60   Input ~ 0
 A-
-Text Label 6500 3350 2    60   ~ 0
-GND
-Text Label 6500 3450 2    60   ~ 0
+Text GLabel 6500 3450 0    60   Input ~ 0
 B-
-Text Label 6500 3550 2    60   ~ 0
+Text GLabel 6500 3550 0    60   Input ~ 0
 B+
-Text Label 6500 3650 2    60   ~ 0
-GND
-Text Label 6500 3850 2    60   ~ 0
+Text GLabel 6500 3850 0    60   Input ~ 0
 +3.3V
-Text Label 6500 3950 2    60   ~ 0
+Text GLabel 6500 3950 0    60   Input ~ 0
 +3.3V
-Text Label 6500 4050 2    60   ~ 0
-GND
-Text Label 6500 4150 2    60   ~ 0
-GND
-Text Label 4250 4150 0    60   ~ 0
-+3.3V
-Text Label 4250 4050 0    60   ~ 0
-GND
-Text Label 4250 3850 0    60   ~ 0
-A+
-Text Label 4250 3750 0    60   ~ 0
-A-
-Text Label 4250 3650 0    60   ~ 0
-GND
-Text Label 4250 3550 0    60   ~ 0
-B-
-Text Label 4250 3450 0    60   ~ 0
-B+
 $Comp
-L CONN_1 P1
-U 1 1 54462EF2
-P 4100 3450
-F 0 "P1" H 4180 3450 40  0000 L CNN
-F 1 "CONN_1" H 4100 3505 30  0001 C CNN
-F 2 "" H 4100 3450 60  0000 C CNN
-F 3 "" H 4100 3450 60  0000 C CNN
-	1    4100 3450
+L CONN1 CN1
+U 1 1 5767D520
+P 3675 3400
+F 0 "CN1" H 4025 3350 60  0000 C CNN
+F 1 "B+" H 3800 3350 60  0000 C CNN
+F 2 "" H 3675 3400 60  0000 C CNN
+F 3 "" H 3675 3400 60  0000 C CNN
+	1    3675 3400
 	-1   0    0    1
 $EndComp
 $Comp
-L CONN_1 P2
-U 1 1 54462F8B
-P 4100 3550
-F 0 "P2" H 4180 3550 40  0000 L CNN
-F 1 "CONN_1" H 4100 3605 30  0001 C CNN
-F 2 "" H 4100 3550 60  0000 C CNN
-F 3 "" H 4100 3550 60  0000 C CNN
-	1    4100 3550
+L CONN1 CN2
+U 1 1 5767DBCF
+P 3675 3500
+F 0 "CN2" H 4025 3450 60  0000 C CNN
+F 1 "B-" H 3800 3450 60  0000 C CNN
+F 2 "" H 3675 3500 60  0000 C CNN
+F 3 "" H 3675 3500 60  0000 C CNN
+	1    3675 3500
 	-1   0    0    1
 $EndComp
 $Comp
-L CONN_1 P3
-U 1 1 54462F91
-P 4100 3650
-F 0 "P3" H 4180 3650 40  0000 L CNN
-F 1 "CONN_1" H 4100 3705 30  0001 C CNN
-F 2 "" H 4100 3650 60  0000 C CNN
-F 3 "" H 4100 3650 60  0000 C CNN
-	1    4100 3650
+L CONN1 CN3
+U 1 1 5767DBF0
+P 3675 3600
+F 0 "CN3" H 4025 3550 60  0000 C CNN
+F 1 "GND" H 3800 3550 60  0000 C CNN
+F 2 "" H 3675 3600 60  0000 C CNN
+F 3 "" H 3675 3600 60  0000 C CNN
+	1    3675 3600
 	-1   0    0    1
 $EndComp
 $Comp
-L CONN_1 P4
-U 1 1 54462F97
-P 4100 3750
-F 0 "P4" H 4180 3750 40  0000 L CNN
-F 1 "CONN_1" H 4100 3805 30  0001 C CNN
-F 2 "" H 4100 3750 60  0000 C CNN
-F 3 "" H 4100 3750 60  0000 C CNN
-	1    4100 3750
+L CONN1 CN4
+U 1 1 5767DC16
+P 3675 3700
+F 0 "CN4" H 4025 3650 60  0000 C CNN
+F 1 "A-" H 3800 3650 60  0000 C CNN
+F 2 "" H 3675 3700 60  0000 C CNN
+F 3 "" H 3675 3700 60  0000 C CNN
+	1    3675 3700
 	-1   0    0    1
 $EndComp
 $Comp
-L CONN_1 P5
-U 1 1 54462F9D
-P 4100 3850
-F 0 "P5" H 4180 3850 40  0000 L CNN
-F 1 "CONN_1" H 4100 3905 30  0001 C CNN
-F 2 "" H 4100 3850 60  0000 C CNN
-F 3 "" H 4100 3850 60  0000 C CNN
-	1    4100 3850
+L CONN1 CN5
+U 1 1 5767DC3F
+P 3675 3800
+F 0 "CN5" H 4025 3750 60  0000 C CNN
+F 1 "A+" H 3800 3750 60  0000 C CNN
+F 2 "" H 3675 3800 60  0000 C CNN
+F 3 "" H 3675 3800 60  0000 C CNN
+	1    3675 3800
 	-1   0    0    1
 $EndComp
 $Comp
-L CONN_1 P6
-U 1 1 54462FA3
-P 4100 4050
-F 0 "P6" H 4180 4050 40  0000 L CNN
-F 1 "CONN_1" H 4100 4105 30  0001 C CNN
-F 2 "" H 4100 4050 60  0000 C CNN
-F 3 "" H 4100 4050 60  0000 C CNN
-	1    4100 4050
+L CONN1 CN6
+U 1 1 5767DC65
+P 3675 3900
+F 0 "CN6" H 4025 3850 60  0000 C CNN
+F 1 "GND" H 3800 3850 60  0000 C CNN
+F 2 "" H 3675 3900 60  0000 C CNN
+F 3 "" H 3675 3900 60  0000 C CNN
+	1    3675 3900
 	-1   0    0    1
 $EndComp
 $Comp
-L CONN_1 P7
-U 1 1 54462FA9
-P 4100 4150
-F 0 "P7" H 4180 4150 40  0000 L CNN
-F 1 "CONN_1" H 4100 4205 30  0001 C CNN
-F 2 "" H 4100 4150 60  0000 C CNN
-F 3 "" H 4100 4150 60  0000 C CNN
-	1    4100 4150
+L CONN1 CN7
+U 1 1 5767DC98
+P 3675 4000
+F 0 "CN7" H 4025 3950 60  0000 C CNN
+F 1 "+3.3V" H 3800 3950 60  0000 C CNN
+F 2 "" H 3675 4000 60  0000 C CNN
+F 3 "" H 3675 4000 60  0000 C CNN
+	1    3675 4000
 	-1   0    0    1
 $EndComp
+Text GLabel 3875 3850 2    60   Input ~ 0
+GND
+Text GLabel 3875 3550 2    60   Input ~ 0
+GND
+Text GLabel 3875 3750 2    60   Input ~ 0
+A+
+Text GLabel 3875 3650 2    60   Input ~ 0
+A-
+Text GLabel 3875 3450 2    60   Input ~ 0
+B-
+Text GLabel 3875 3350 2    60   Input ~ 0
+B+
+Text GLabel 3875 3950 2    60   Input ~ 0
++3.3V
 $EndSCHEMATC

Commit message: final
for now
Parts:
- CN1, CN2, CN3, CN4, CN5, CN6, CN7: footprint (none) -> eeepc_ssd:CONN1
- CN8: footprint (none) -> eeepc_ssd:uSATA
Changed lines of the file:
@@
 LIBS:valves
 LIBS:eeepc_ssd
+LIBS:uSATAboard-cache
 EELAYER 25 0
 EELAYER END
@@
 F 0 "CN8" H 6875 3050 60  0000 C CNN
 F 1 "USATA" H 7325 1125 60  0000 C CNN
-F 2 "" H 6800 3000 60  0000 C CNN
+F 2 "eeepc_ssd:uSATA" H 6800 3000 60  0001 C CNN
 F 3 "" H 6800 3000 60  0000 C CNN
 	1    6800 3000
@@
 F 0 "CN1" H 4025 3350 60  0000 C CNN
 F 1 "B+" H 3800 3350 60  0000 C CNN
-F 2 "" H 3675 3400 60  0000 C CNN
+F 2 "eeepc_ssd:CONN1" H 3675 3400 60  0001 C CNN
 F 3 "" H 3675 3400 60  0000 C CNN
 	1    3675 3400
@@
 F 0 "CN2" H 4025 3450 60  0000 C CNN
 F 1 "B-" H 3800 3450 60  0000 C CNN
-F 2 "" H 3675 3500 60  0000 C CNN
+F 2 "eeepc_ssd:CONN1" H 3675 3500 60  0001 C CNN
 F 3 "" H 3675 3500 60  0000 C CNN
 	1    3675 3500
@@
 F 0 "CN3" H 4025 3550 60  0000 C CNN
 F 1 "GND" H 3800 3550 60  0000 C CNN
-F 2 "" H 3675 3600 60  0000 C CNN
+F 2 "eeepc_ssd:CONN1" H 3675 3600 60  0001 C CNN
 F 3 "" H 3675 3600 60  0000 C CNN
 	1    3675 3600
@@
 F 0 "CN4" H 4025 3650 60  0000 C CNN
 F 1 "A-" H 3800 3650 60  0000 C CNN
-F 2 "" H 3675 3700 60  0000 C CNN
+F 2 "eeepc_ssd:CONN1" H 3675 3700 60  0001 C CNN
 F 3 "" H 3675 3700 60  0000 C CNN
 	1    3675 3700
@@
 F 0 "CN5" H 4025 3750 60  0000 C CNN
 F 1 "A+" H 3800 3750 60  0000 C CNN
-F 2 "" H 3675 3800 60  0000 C CNN
+F 2 "eeepc_ssd:CONN1" H 3675 3800 60  0001 C CNN
 F 3 "" H 3675 3800 60  0000 C CNN
 	1    3675 3800
@@
 F 0 "CN6" H 4025 3850 60  0000 C CNN
 F 1 "GND" H 3800 3850 60  0000 C CNN
-F 2 "" H 3675 3900 60  0000 C CNN
+F 2 "eeepc_ssd:CONN1" H 3675 3900 60  0001 C CNN
 F 3 "" H 3675 3900 60  0000 C CNN
 	1    3675 3900
@@
 F 0 "CN7" H 4025 3950 60  0000 C CNN
 F 1 "+3.3V" H 3800 3950 60  0000 C CNN
-F 2 "" H 3675 4000 60  0000 C CNN
+F 2 "eeepc_ssd:CONN1" H 3675 4000 60  0001 C CNN
 F 3 "" H 3675 4000 60  0000 C CNN
 	1    3675 4000
